File: schematics/landrumower/landrumower.kicad_pcb (KiCad board)
At the start: 2 copper layers, 99 x 90 mm, 30 parts, among them J1 UART, J10 Lift, J11 MotorLeft, J12 Conn_01x06_Female, J13 Conn_01x06_Female, J14 Rain, J15 MotorMow, J16 Conn_01x06_Female, J17 Conn_01x06_Female, J18 StopButton, J19 ReserveGPIO, J2 I2C0, J20 ResrveGPIO/ADC0, J21 ReserveGPIO/ADC1, J3 Power, J4 I2C1, J5 BumperX, J6 MotorRight, J7 Conn_01x06_Female, J8 Conn_01x06_Female, J9 BumperY, U1 Pico

Commit message: Update schematics for landrumower pcb
Parts:
- removed the REF** at (103.0, 118.0)
- removed the REF** at (192.3, 37.6)
- removed the REF** at (103.0, 38.0)
- removed the REF** at (192.3, 118.4)
- added C2: C_Small, Capacitor_SMD:C_0805_2012Metric_Pad1.18x1.45mm_HandSolder, F.Cu at (166.0, 114.0)
- added J22: IMU, Connector_PinSocket_2.54mm:PinSocket_1x08_P2.54mm_Vertical, F.Cu at (124.9, 61.0)
- added J23: IN+, Connector_PinSocket_2.54mm:PinSocket_1x01_P2.54mm_Vertical, F.Cu at (185.0, 142.0)
- added J24: I2C reserve0, Connector_JST:JST_EH_B4B-EH-A_1x04_P2.50mm_Vertical, F.Cu at (126.5, 80.4)
- added J25: I2C reserve1, Connector_JST:JST_EH_B4B-EH-A_1x04_P2.50mm_Vertical, F.Cu at (126.5, 71.4)
- added J26: OUT+, Connector_PinSocket_2.54mm:PinSocket_1x01_P2.54mm_Vertical, F.Cu at (145.5, 142.0)
- added J27: IN-, Connector_PinSocket_2.54mm:PinSocket_1x01_P2.54mm_Vertical, F.Cu at (185.0, 124.8)
- added J28: OUT-, Connector_PinSocket_2.54mm:PinSocket_1x01_P2.54mm_Vertical, F.Cu at (145.5, 124.8)
- added JP1: I2C adress, Connector_PinHeader_2.54mm:PinHeader_1x03_P2.54mm_Vertical, F.Cu at (149.0, 63.5)
- added R4: 100k, Resistor_SMD:R_0805_2012Metric_Pad1.20x1.40mm_HandSolder, F.Cu at (92.0, 111.0)
- added R5: 100k, Resistor_SMD:R_0805_2012Metric_Pad1.20x1.40mm_HandSolder, F.Cu at (73.0, 111.0)
- added R6: 100k, Resistor_SMD:R_0805_2012Metric_Pad1.20x1.40mm_HandSolder, F.Cu at (111.0, 111.0)
- added REF**: MountingHole_2.7mm, MountingHole:MountingHole_2.7mm, F.Cu at (157.0, 60.0)
- added REF**: MountingHole_2.7mm, MountingHole:MountingHole_2.7mm, F.Cu at (215.0, 109.0)
- added REF**: MountingHole_4.3mm_M4, MountingHole:MountingHole_4.3mm_M4, F.Cu at (54.0, 50.0)
- added REF**: MountingHole_2.7mm, MountingHole:MountingHole_2.7mm, F.Cu at (215.0, 60.0)
- added REF**: MountingHole_4.3mm_M4, MountingHole:MountingHole_4.3mm_M4, F.Cu at (54.0, 140.0)
- added REF**: MountingHole_4.3mm_M4, MountingHole:MountingHole_4.3mm_M4, F.Cu at (214.0, 50.0)
- added REF**: MountingHole_4.3mm_M4, MountingHole:MountingHole_4.3mm_M4, F.Cu at (214.0, 140.0)
- added REF**: MountingHole_2.7mm, MountingHole:MountingHole_2.7mm, F.Cu at (157.0, 109.0)
- added U2: Raspberry_Pi_2_3, Connector_PinSocket_2.54mm:PinSocket_2x20_P2.54mm_Vertical, F.Cu at (161.9, 107.7)
- J1: value UART -> MotorRight; footprint Connector_JST:JST_EH_B3B-EH-A_1x03_P2.50mm_Vertical -> Connector_JST:JST_EH_B6B-EH-A_1x06_P2.50mm_Vertical
- J10: value Lift -> Conn_01x06_Female; footprint Connector_JST:JST_EH_B3B-EH-A_1x03_P2.50mm_Vertical -> Connector_PinSocket_2.54mm:PinSocket_1x06_P2.54mm_Vertical
- J11: value MotorLeft -> UART; footprint Connector_JST:JST_EH_B6B-EH-A_1x06_P2.50mm_Vertical -> Connector_JST:JST_EH_B3B-EH-A_1x03_P2.50mm_Vertical
- J12: value Conn_01x06_Female -> BumperY; footprint Connector_PinSocket_2.54mm:PinSocket_1x06_P2.54mm_Vertical -> Connector_JST:JST_EH_B3B-EH-A_1x03_P2.50mm_Vertical
- J13: value Conn_01x06_Female -> BumperX; footprint Connector_PinSocket_2.54mm:PinSocket_1x06_P2.54mm_Vertical -> Connector_JST:JST_EH_B3B-EH-A_1x03_P2.50mm_Vertical
- J14: value Rain -> I2C0; footprint Connector_JST:JST_EH_B3B-EH-A_1x03_P2.50mm_Vertical -> Connector_JST:JST_EH_B4B-EH-A_1x04_P2.50mm_Vertical
- J15: value MotorMow -> Lift; footprint Connector_JST:JST_EH_B6B-EH-A_1x06_P2.50mm_Vertical -> Connector_JST:JST_EH_B3B-EH-A_1x03_P2.50mm_Vertical
- J16: value Conn_01x06_Female -> StopButton; footprint Connector_PinSocket_2.54mm:PinSocket_1x06_P2.54mm_Vertical -> Connector_JST:JST_EH_B3B-EH-A_1x03_P2.50mm_Vertical
- J17: value Conn_01x06_Female -> I2C1; footprint Connector_PinSocket_2.54mm:PinSocket_1x06_P2.54mm_Vertical -> Connector_JST:JST_EH_B4B-EH-A_1x04_P2.50mm_Vertical
- J18: value StopButton -> Rain
- J19: value ReserveGPIO -> ResrveGPIO/ADC0
- J2: value I2C0 -> Conn_01x06_Female; footprint Connector_JST:JST_EH_B4B-EH-A_1x04_P2.50mm_Vertical -> Connector_PinSocket_2.54mm:PinSocket_1x06_P2.54mm_Vertical
- J20: value ResrveGPIO/ADC0 -> ReserveGPIO
- J3: footprint Connector_JST:JST_EH_B2B-EH-A_1x02_P2.50mm_Vertical -> TerminalBlock:TerminalBlock_Altech_AK300-2_P5.00mm
- J4: value I2C1 -> Conn_01x06_Female; footprint Connector_JST:JST_EH_B4B-EH-A_1x04_P2.50mm_Vertical -> Connector_PinSocket_2.54mm:PinSocket_1x06_P2.54mm_Vertical
- J5: value BumperX -> MotorLeftt; footprint Connector_JST:JST_EH_B3B-EH-A_1x03_P2.50mm_Vertical -> Connector_JST:JST_EH_B6B-EH-A_1x06_P2.50mm_Vertical
- J6: value MotorRight -> Conn_01x06_Female; footprint Connector_JST:JST_EH_B6B-EH-A_1x06_P2.50mm_Vertical -> Connector_PinSocket_2.54mm:PinSocket_1x06_P2.54mm_Vertical
- J8: value Conn_01x06_Female -> MotorMow; footprint Connector_PinSocket_2.54mm:PinSocket_1x06_P2.54mm_Vertical -> Connector_JST:JST_EH_B6B-EH-A_1x06_P2.50mm_Vertical
- J9: value BumperY -> Conn_01x06_Female; footprint Connector_JST:JST_EH_B3B-EH-A_1x03_P2.50mm_Vertical -> Connector_PinSocket_2.54mm:PinSocket_1x06_P2.54mm_Vertical
- moved J5 139.9 mm to (64.8, 139.7)
- moved J3 131.0 mm to (196.2, 138.0)
- moved J2 121.0 mm to (59.7, 107.0), turned to 90 degrees
- moved J18 116.4 mm to (55.3, 61.5), turned to -90 degrees
- moved J1 110.2 mm to (87.8, 139.7)
- moved J10 107.5 mm to (97.7, 117.0), turned to 90 degrees
- moved J4 102.0 mm to (78.7, 117.0), turned to 90 degrees
- moved J9 98.6 mm to (97.7, 107.0), turned to 90 degrees
- moved J19 88.1 mm to (71.3, 61.5), turned to -90 degrees
- moved J11 85.9 mm to (191.0, 49.0)
- moved J21 83.6 mm to (63.3, 61.5), turned to -90 degrees
- moved J15 80.3 mm to (95.3, 61.5), turned to -90 degrees
- moved J16 74.9 mm to (87.3, 61.5), turned to -90 degrees
- moved C1 59.1 mm to (60.0, 83.0), turned to 0 degrees
- moved U1 58.1 mm to (83.0, 88.0)
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Connections:
- J1 pad 1: UART (TX) -> +5V
- J1 pad 2: GND -> Net-(J1-Pad2)
- J1 pad 3: UART (RX) -> Net-(J1-Pad3)
- J10 pad 1: +3V3 -> Net-(J10-Pad1)
- J10 pad 2: lift -> Net-(J10-Pad2)
- J11 pad 1: +5V -> UART (PI:RX PICO:TX)
- J11 pad 2: Net-(J11-Pad2) -> GND
- J11 pad 3: Net-(J11-Pad3) -> UART (PI:TX PICO:RX)
- J12 pad 1: pinMotorLeftImp -> +3V3
- J12 pad 2: pinMotorLeftPWM -> bumperY
- J13 pad 1: Net-(J11-Pad2) -> +3V3
- J13 pad 2: Net-(J11-Pad3) -> bumperX
- J14 pad 2: rain -> I2C0 (SDA)
- J14 pad 3: GND -> I2C0 (SCL)
- J15 pad 1: +5V -> +3V3
- J15 pad 2: Net-(J15-Pad2) -> lift
- J15 pad 3: Net-(J15-Pad3) -> GND
- J16 pad 1: pinMotorMowImp -> +3V3
- J16 pad 2: pinMotorMowPWM -> stopButton
- J17 pad 1: Net-(J15-Pad2) -> +3V3
- J17 pad 2: Net-(J15-Pad3) -> I2C1 (SDA)
- J17 pad 3: GND -> I2C1 (SCL)
- J17 pad 4: +5V -> GND
- J18 pad 2: stopButton -> rain
- J19 pad 2: reserve GPIO -> reserve GPIO/ADC 0
- J2 pad 1: +3V3 -> pinMotorRightImp
- J2 pad 2: I2C0 (SDA) -> pinMotorRightPWM
- J2 pad 3: I2C0 (SCL) -> GND
- J2 pad 4: GND -> +3V3
- J20 pad 2: reserve GPIO/ADC 0 -> reserve GPIO
- J3 pad 2: +5V -> +24V
- J4 pad 1: +3V3 -> Net-(J1-Pad2)
- J4 pad 2: I2C1 (SDA) -> Net-(J1-Pad3)
- J4 pad 3: I2C1 (SCL) -> GND
- J4 pad 4: GND -> +5V
- J5 pad 1: +3V3 -> +5V
- J5 pad 2: bumperX -> Net-(J5-Pad2)
- J5 pad 3: GND -> Net-(J5-Pad3)
- J6 pad 1: +5V -> pinMotorLeftImp
- J6 pad 2: Net-(J6-Pad2) -> pinMotorLeftPWM
- J6 pad 3: Net-(J6-Pad3) -> GND
- J6 pad 4: Net-(J6-Pad4) -> +3V3
- J6 pad 5: Net-(J6-Pad5) -> pinMotorLeftDir
- J6 pad 6: GND -> pinMotorLeftBrake
- J7 pad 1: pinMotorRightImp -> Net-(J5-Pad2)
- J7 pad 2: pinMotorRightPWM -> Net-(J5-Pad3)
- J7 pad 4: +3V3 -> +5V
- J7 pad 5: pinMotorRightDir -> Net-(J5-Pad4)
- J7 pad 6: pinMotorRightBrake -> Net-(J5-Pad5)
- J8 pad 1: Net-(J6-Pad2) -> +5V
- J8 pad 2: Net-(J6-Pad3) -> Net-(J10-Pad1)
- J8 pad 3: GND -> Net-(J10-Pad2)
- J8 pad 4: +5V -> Net-(J10-Pad5)
- J8 pad 5: Net-(J6-Pad4) -> Net-(J10-Pad6)
- J8 pad 6: Net-(J6-Pad5) -> GND
- J9 pad 1: +3V3 -> pinMotorMowImp
- J9 pad 2: bumperY -> pinMotorMowPWM
- U1 pad 1: UART (TX) -> UART (PI:RX PICO:TX)
- U1 pad 2: UART (RX) -> UART (PI:TX PICO:RX)
- U1 pad 31: reserve GPIO/ADC 1 -> reserve GPIO/ADC 0
- U1 pad 32: reserve GPIO/ADC 0 -> reserve GPIO/ADC 1
Routing:
- net UART (PI:RX PICO:TX): track 0.00 -> 206.2 mm
- net UART (PI:TX PICO:RX): track 0.00 -> 204.4 mm
- net +5V: track 183.1 -> 344.1 mm
- net +3V3: track 289.5 -> 191.4 mm
- net I2C(SCL): track 0.00 -> 72.6 mm
- net I2C(SDA): track 0.00 -> 65.1 mm
- net UART (RX): track 59.6 -> 0.00 mm
- net UART (TX): track 55.1 -> 0.00 mm
- net Net-(J10-Pad6): track 0.00 -> 33.2 mm
- net Net-(J1-Pad5): track 0.00 -> 31.5 mm
- net Net-(J5-Pad5): track 0.00 -> 29.8 mm
- net Net-(J10-Pad1): track 0.00 -> 29.2 mm
- net Net-(J10-Pad2): track 0.00 -> 29.2 mm
- net Net-(J1-Pad2): track 0.00 -> 27.5 mm
- net Net-(J1-Pad3): track 0.00 -> 27.5 mm
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Other:
- board size 99 x 90 mm -> 170 x 100 mm
- board text added: "Landrumower PCB V1.0"

Commit message: PCB changes for Landrumower
Parts:
- added J29: RPI GPIOs1, Connector_JST:JST_EH_B6B-EH-A_1x06_P2.50mm_Vertical, F.Cu at (162.8, 49.0)
- added J30: RPI GPIOs2, Connector_JST:JST_EH_B6B-EH-A_1x06_P2.50mm_Vertical, F.Cu at (183.0, 49.0)
- added TP1: TP_5V, TestPoint:TestPoint_Pad_D2.0mm, B.Cu at (125.0, 49.0)
- added TP2: TP3.3V, TestPoint:TestPoint_Pad_D2.0mm, B.Cu at (130.0, 49.0)
- added TP3: TP_GND, TestPoint:TestPoint_Pad_D2.0mm, B.Cu at (135.0, 49.0)
- added kibuzzard-65CA0A0A: G***, kibuzzard-65CA0A0A, F.Cu at (71.3, 142.9)
- added kibuzzard-65CA0A31: G***, kibuzzard-65CA0A31, F.Cu at (94.3, 142.9)
- added kibuzzard-65CA0A42: G***, kibuzzard-65CA0A42, F.Cu at (117.4, 142.8)
- added kibuzzard-65CA0A7B: G***, kibuzzard-65CA0A7B, F.Cu at (77.3, 135.1)
- added kibuzzard-65CA0A7B: G***, kibuzzard-65CA0A7B, F.Cu at (123.3, 135.1)
- added kibuzzard-65CA0A7B: G***, kibuzzard-65CA0A7B, F.Cu at (100.3, 135.1)
- added kibuzzard-65CA0AF1: G***, kibuzzard-65CA0AF1, F.Cu at (74.8, 133.5)
- added kibuzzard-65CA0AF1: G***, kibuzzard-65CA0AF1, F.Cu at (97.7, 133.5)
- added kibuzzard-65CA0AF1: G***, kibuzzard-65CA0AF1, F.Cu at (120.8, 133.5)
- added kibuzzard-65CA0B61: G***, kibuzzard-65CA0B61, F.Cu at (95.3, 134.0)
- added kibuzzard-65CA0B61: G***, kibuzzard-65CA0B61, F.Cu at (118.3, 134.0)
- added kibuzzard-65CA0BDD: G***, kibuzzard-65CA0BDD, F.Cu at (72.3, 134.0)
- added kibuzzard-65CA0BE5: G***, kibuzzard-65CA0BE5, F.Cu at (69.7, 133.9)
- added kibuzzard-65CA0BE5: G***, kibuzzard-65CA0BE5, F.Cu at (115.8, 134.0)
- added kibuzzard-65CA0BE5: G***, kibuzzard-65CA0BE5, F.Cu at (92.8, 134.0)
- added kibuzzard-65CA0CDE: G***, kibuzzard-65CA0CDE, F.Cu at (90.3, 134.0)
- added kibuzzard-65CA0CDE: G***, kibuzzard-65CA0CDE, F.Cu at (113.3, 134.0)
- added kibuzzard-65CA0CDE: G***, kibuzzard-65CA0CDE, F.Cu at (67.2, 134.0)
- added kibuzzard-65CA0D25: G***, kibuzzard-65CA0D25, F.Cu at (64.7, 135.4)
- added kibuzzard-65CA0D25: G***, kibuzzard-65CA0D25, F.Cu at (110.7, 135.4)
- added kibuzzard-65CA0D25: G***, kibuzzard-65CA0D25, F.Cu at (87.8, 135.4)
- added kibuzzard-65CA1367: G***, kibuzzard-65CA1367, F.Cu at (126.3, 103.2)
- added kibuzzard-65CA1367: G***, kibuzzard-65CA1367, F.Cu at (126.3, 94.0)
- added kibuzzard-65CA137E: G***, kibuzzard-65CA137E, F.Cu at (131.2, 103.0)
- added kibuzzard-65CA137E: G***, kibuzzard-65CA137E, F.Cu at (132.5, 63.2)
- added kibuzzard-65CA137E: G***, kibuzzard-65CA137E, F.Cu at (131.2, 93.8)
- added kibuzzard-65CA1392: G***, kibuzzard-65CA1392, F.Cu at (128.9, 93.8)
- added kibuzzard-65CA1392: G***, kibuzzard-65CA1392, F.Cu at (128.9, 103.0)
- added kibuzzard-65CA1392: G***, kibuzzard-65CA1392, F.Cu at (130.1, 63.2)
- added kibuzzard-65CA13E2: G***, kibuzzard-65CA13E2, F.Cu at (133.7, 103.0)
- added kibuzzard-65CA13E2: G***, kibuzzard-65CA13E2, F.Cu at (133.7, 93.8)
- added kibuzzard-65CA13E2: G***, kibuzzard-65CA13E2, F.Cu at (127.5, 63.1)
- added kibuzzard-65CA1528: G***, kibuzzard-65CA1528, F.Cu at (125.0, 63.3)
- added kibuzzard-65CA15BA: G***, kibuzzard-65CA15BA, F.Cu at (107.9, 64.0)
- added kibuzzard-65CA15CC: G***, kibuzzard-65CA15CC, F.Cu at (107.9, 66.5)
- added kibuzzard-65CA15DA: G***, kibuzzard-65CA15DA, F.Cu at (108.0, 61.5)
- added kibuzzard-65CA18B9: G***, kibuzzard-65CA18B9, F.Cu at (183.0, 52.6)
- added kibuzzard-65CA18B9: G***, kibuzzard-65CA18B9, F.Cu at (162.7, 52.6)
- added kibuzzard-65CA18EE: G***, kibuzzard-65CA18EE, F.Cu at (185.6, 53.1)
- added kibuzzard-65CA18EE: G***, kibuzzard-65CA18EE, F.Cu at (165.3, 53.1)
- added kibuzzard-65CA190F: G***, kibuzzard-65CA190F, F.Cu at (167.8, 53.3)
- added kibuzzard-65CA191B: G***, kibuzzard-65CA191B, F.Cu at (170.3, 53.3)
- added kibuzzard-65CA1927: G***, kibuzzard-65CA1927, F.Cu at (172.8, 53.3)
- added kibuzzard-65CA193C: G***, kibuzzard-65CA193C, F.Cu at (195.6, 52.8)
- added kibuzzard-65CA193C: G***, kibuzzard-65CA193C, F.Cu at (175.3, 52.9)
- added kibuzzard-65CA19E7: G***, kibuzzard-65CA19E7, F.Cu at (188.1, 53.3)
- added kibuzzard-65CA19F9: G***, kibuzzard-65CA19F9, F.Cu at (190.6, 53.5)
- added kibuzzard-65CA1A09: G***, kibuzzard-65CA1A09, F.Cu at (193.1, 53.5)
- J20: value ReserveGPIO -> PowerPCB; footprint Connector_JST:JST_EH_B3B-EH-A_1x03_P2.50mm_Vertical -> Connector_JST:JST_EH_B5B-EH-A_1x05_P2.50mm_Vertical
- moved J11 41.5 mm to (149.5, 49.0)
- moved J20 31.0 mm to (107.7, 49.0), turned to 0 degrees
- moved J23 12.5 mm to (172.5, 141.0)
- moved J26 12.5 mm to (133.0, 141.0)
- moved J27 12.5 mm to (172.5, 123.8)
- moved J28 12.5 mm to (133.0, 123.8)
- moved J12 8.00 mm to (95.3, 61.5)
- moved J13 8.00 mm to (103.3, 61.5)
- moved J15 8.00 mm to (87.3, 61.5)
- moved J16 8.00 mm to (79.3, 61.5)
- moved J22 5.30 mm to (124.9, 66.3)
- moved J3 3.00 mm to (199.2, 138.0)
- moved C1 1.00 mm to (60.0, 82.0)
Connections:
- J14 pad 2: I2C0 (SDA) -> I2C0 (SCL)
- J14 pad 3: I2C0 (SCL) -> I2C0 (SDA)
- J17 pad 2: I2C1 (SDA) -> I2C1 (SCL)
- J17 pad 3: I2C1 (SCL) -> I2C1 (SDA)
- J20 pad 2: reserve GPIO -> I2C0 (SDA)
- J20 pad 3: GND -> I2C0 (SCL)
- U1 pad 29: reserve GPIO -> pinBatterySwitch
- U2 pad 1: unconnected-(U2-Pad1) -> +3.3VP
- U2 pad 17: unconnected-(U2-Pad17) -> +3.3VP
- U2 pad 27: unconnected-(U2-Pad27) -> GPIO1
- U2 pad 28: unconnected-(U2-Pad28) -> GPIO2
- U2 pad 29: unconnected-(U2-Pad29) -> GPIO5
- U2 pad 31: unconnected-(U2-Pad31) -> GPIO6
- U2 pad 33: unconnected-(U2-Pad33) -> GPIO13
- U2 pad 35: unconnected-(U2-Pad35) -> GPIO19
- U2 pad 7: unconnected-(U2-Pad7) -> GPIO4
Routing:
- net +3.3VP: track 0.00 -> 99.9 mm
- net GPIO2: track 0.00 -> 72.5 mm
- net GPIO5: track 0.00 -> 68.9 mm
- net GPIO1: track 0.00 -> 68.9 mm
- net pinBatterySwitch: track 0.00 -> 68.6 mm
- net GPIO19: track 0.00 -> 63.7 mm
- net GPIO13: track 0.00 -> 63.7 mm
- net GPIO6: track 0.00 -> 63.7 mm
- net +5V: track 344.1 -> 385.2 mm
- net I2C0 (SDA): track 30.9 -> 67.3 mm
- net +3V3: track 191.4 -> 221.2 mm
- net I2C0 (SCL): track 36.6 -> 62.0 mm
- net reserve GPIO: track 18.2 -> 0.00 mm
- net GND: track 0.00 -> 18.2 mm
- net +24V: track 17.9 -> 34.6 mm
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Other:
- board text added: "+"
- board text added: "-"
- board text added: "24V"
- board text added: "BumperX"
- board text added: "BumperY"
- board text added: "DC/DC step down converter"
- board text added: "I2C address"
- board text added: "I2C reserve 0"
- board text added: "I2C reserve 1"
- board text added: "I2C0"
- board text added: "I2C1"
- board text added: "IMU"
- board text added: "IN+"
- board text added: "IN-"
- board text added: "Lift"
- board text added: "OUT+"
- board text added: "OUT-"
- board text added: "PowerPCB"
- board text added: "RPi GPIOs1"
- board text added: "RPi GPIOs2"
- board text added: "Rain"
- board text added: "Raspberry PI"
- board text added: "Raspberry Pi Pico"
- board text added: "ReserveGPIO/ADC0"
- board text added: "ReserveGPIO/ADC1"
- board text added: "StopButton"
- board text added: "UART"

Commit message: Update schematics
Parts:
- removed kibuzzard-65CA0A0A: G***, kibuzzard-65CA0A0A
- removed kibuzzard-65CA0A31: G***, kibuzzard-65CA0A31
- removed kibuzzard-65CA0A42: G***, kibuzzard-65CA0A42
- removed the kibuzzard-65CA13E2 at (133.7, 103.0)
- removed the kibuzzard-65CA13E2 at (133.7, 93.8)
- added kibuzzard-65CA34CF: G***, kibuzzard-65CA34CF, F.Cu at (149.0, 54.0)
- added kibuzzard-65CA34D8: G***, kibuzzard-65CA34D8, F.Cu at (144.0, 54.0)
- added kibuzzard-65CA3687: G***, kibuzzard-65CA3687, F.Cu at (93.3, 52.7)
- added kibuzzard-65CA369C: G***, kibuzzard-65CA369C, F.Cu at (95.8, 54.0)
- added kibuzzard-65CA36D0: G***, kibuzzard-65CA36D0, F.Cu at (98.4, 54.0)
- added kibuzzard-65CA3704: G***, kibuzzard-65CA3704, F.Cu at (100.8, 53.9)
- added kibuzzard-65CA3716: G***, kibuzzard-65CA3716, F.Cu at (103.4, 52.5)
- moved JP1 77.4 mm to (137.1, 140.0), turned to -90 degrees
- moved J22 57.0 mm to (140.9, 121.0), turned to -90 degrees
- moved J23 28.8 mm to (201.3, 141.3)
- moved J26 28.8 mm to (161.8, 141.3)
- moved J27 28.8 mm to (201.3, 124.1)
- moved J28 28.8 mm to (161.8, 124.1)
- moved C2 16.0 mm to (150.2, 116.5)
- moved REF** 16.0 mm to (141.2, 62.5)
- moved REF** 16.0 mm to (199.2, 111.5)
- moved REF** 16.0 mm to (199.2, 62.5)
- moved REF** 16.0 mm to (141.2, 111.5)
- moved U2 16.0 mm to (146.1, 110.2)
- moved J3 15.7 mm to (212.4, 129.4), turned to 90 degrees
- moved J20 14.4 mm to (93.3, 48.8)
- moved TP1 14.4 mm to (110.6, 48.8)
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Routing:
- net +5V: track 385.2 -> 425.5 mm
- net I2C(SDA): track 59.8 -> 93.7 mm
- net GND: track 18.2 -> 0.00 mm
- net pinBatterySwitch: track 68.6 -> 52.2 mm
- net UART (PI:TX PICO:RX): track 202.7 -> 215.9 mm
- net +24V: track 34.6 -> 21.5 mm
- net UART (PI:RX PICO:TX): track 204.5 -> 191.8 mm
- net I2C0 (SDA): track 67.3 -> 56.3 mm
- net Net-(J22-Pad7): track 11.9 -> 22.7 mm
- net I2C1 (SCL): track 25.4 -> 15.1 mm
- net I2C1 (SDA): track 29.7 -> 21.8 mm
- net +3V3: track 221.2 -> 214.1 mm
- net I2C(SCL): track 67.3 -> 71.2 mm
- net +3.3VP: track 99.9 -> 102.7 mm
- net GPIO5: track 68.9 -> 67.1 mm
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Other:
- outline, holes or cut-outs redrawn
- board text added: "IMU I2C address"
- board text added: "MotorLeft"
- board text added: "MotorMow"
- board text added: "MotorRight"
- board text removed: "I2C address"

Commit message: changes in schematics
Parts:
- added JP2: Jumper_2_Open, Jumper:SolderJumper-2_P1.3mm_Open_Pad1.0x1.5mm, B.Cu at (161.0, 134.0)
- added REF**: OSHW-Logo_7.5x8mm_SilkScreen, Symbol:OSHW-Logo_7.5x8mm_SilkScreen, B.Cu at (178.0, 139.0)
- added REF**: WEEE-Logo_4.2x6mm_SilkScreen, Symbol:WEEE-Logo_4.2x6mm_SilkScreen, B.Cu at (186.0, 139.0)
- added REF**: RoHS-Logo_6mm_SilkScreen, Symbol:RoHS-Logo_6mm_SilkScreen, B.Cu at (185.0, 131.0)
- added REF**: ESD-Logo_6.6x6mm_SilkScreen, Symbol:ESD-Logo_6.6x6mm_SilkScreen, B.Cu at (193.0, 139.0)
- moved C1 8.00 mm to (60.0, 74.0)
Connections:
- J26 pad 1: +5V -> Net-(J26-Pad1)
Routing:
- net +5V: track 425.5 -> 417.3 mm
- net Net-(J26-Pad1): track 0.00 -> 7.05 mm
